File: KiCad/FairberryMainboard/FairberryMainboard.kicad_pcb (KiCad board)
At the start: 2 copper layers, 37.3 x 14.7 mm, 15 parts, among them J1 USB_Header, J2 Conn_02x03_Odd_Even, J4 Conn_01x02, U1 ATmega32U4-MU, U2 BBQ10KBD, Y1 Crystal_GND24

Commit message: Finalisation of v0.3.0 PCB
Parts:
- renumbered J4 to ?
Other:
- board text added: "07.03.2024 Fairberry v0.3.0 ©Dakkaron, 2024"
- board text removed: "14.02.2024 Fairberry v0.3.0 ©Dakkaron, 2024"
Changed lines of the file:
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@@
       (drillshape 0)
       (scaleselection 1)
-      (outputdirectory "gerber")
+      (outputdirectory "gerber/")
     )
   )
@@
     (property "Sheetname" "")
     (attr exclude_from_pos_files)
-    (fp_text reference "J4" (at -3.8 -0.4 90) (layer "F.SilkS")
+    (fp_text reference "" (at -3.8 -0.4 90) (layer "F.SilkS") hide
       (effects (font (size 1 1) (thickness 0.15)))
     )
@@
     (effects (font (size 1.5 1.5) (thickness 0.3)) (justify mirror))
   )
-  (gr_text "14.02.2024\nFairberry\nv0.3.0\n©Dakkaron, 2024" (at 191.15 87.9) (layer "B.SilkS")
+  (gr_text "07.03.2024\nFairberry\nv0.3.0\n©Dakkaron, 2024" (at 191.15 87.9) (layer "B.SilkS")
     (effects (font (size 1.5 1.5) (thickness 0.3)) (justify left mirror))
   )
@@
         (xy 192 97)
         (xy 153.5 97)
-        (xy 153.5 97)
         (xy 153.5 88)
